File: Esquematico_final_KiCad/VW_ServMode_4taGen/VW_ServMode_4taGen.kicad_sch (KiCad schematic)
At the start: 25 parts, among them J1 MicroSDReader, J2 Conn_01x02, J3 ClampConnections, J4 uC_custom, SW1 SW_In, SW2 SW_Out, SW3 SW_Reset

Commit message: Proyecto final actualizado
Parts:
- removed AFF1: LTS-6960HR, Display_7Segment:7SegmentLED_LTS6760_LTS6780, symbol Display_Character:LTS-6960HR
- removed J2: Conn_01x02, symbol Connector_Generic:Conn_01x02
- added AFF2: LTS-6980HR, Display_7Segment:7SegmentLED_LTS6760_LTS6780, symbol Display_Character:LTS-6980HR
- added D7: LED_BAT0, symbol Device:LED
- added D8: LED_ModServOn, symbol Device:LED
- added D9: LED_ModServOff, symbol Device:LED
- added J2: USB-C, symbol Connector_Generic:Conn_01x04
- added J5: TP4056_Custom_2extraOutputs, symbol Connector_Generic:Conn_02x04_Counter_Clockwise
- added J6: 3v3Switch, symbol Connector_Generic:Conn_01x03
- added R12, R13, R14: 330, symbol Device:R
- D1: value LED_B25 -> LED_BAT25
- D2: value LED_B50 -> LED_BAT50
- D3: value LED_B75 -> LED_BAT75
- D4: value LED_B99 -> LED_BAT99
Connections:
- net RESET_A is gone; now on net SWDIO: J4.26 (Pin_26)
- net RESET_B is gone; now on net SWDCLK: J4.25 (Pin_25)
- net +3.3V: now also J4.28 (Pin_28), J6.2 (Pin_2); no longer J3.8 (Pin_8), J4.29 (Pin_29), R1.1, R10.1, R11.1
- net GND: now also R1.1, J5.7 (Pin_7), R12.2, R13.2, R14.2
- net LED_A: now also AFF2.7 (a)
- net LED_B: now also AFF2.6 (b)
- net LED_C: now also AFF2.4 (c)
- net LED_D: now also AFF2.2 (d)
- net LED_E: now also AFF2.1 (e)
- net LED_ERROR: now also J4.20 (Pin_20); no longer J4.15 (Pin_15)
- net LED_F: now also AFF2.9 (f)
- net LED_G: now also AFF2.10 (g)
- net LED_OK: now also J4.19 (Pin_19); no longer J4.14 (Pin_14)
- net SWDCLK: no longer J4.27 (Pin_27)
- net SWDIO: no longer J4.28 (Pin_28)
- net DI_CHARGED: now reaches J4.16 (Pin_16)
- net DI_CHARGED: now also J5.3 (Pin_3)
- net LED_ModServOn: now reaches J4.17 (Pin_17)
- net LED_ModServOn: now also D8.2 (A)
- net LED_ModServOff: now reaches J4.18 (Pin_18)
- net LED_ModServOff: now also D9.2 (A)
- net at R1.2: now also AFF2.8 (C.K.)
- net DO_5V renamed DO_WIRE5V
- net DO_WIRE5V: now also J6.3 (Pin_3)
- net LED_25 renamed LED_B0
- net LED_B0: now also D7.2 (A); no longer D1.2 (A)
- net LED_50 renamed LED_B25
- net LED_B25: now also D1.2 (A); no longer D2.2 (A)
- net LED_75 renamed LED_B50
- net LED_B50: now also D2.2 (A); no longer D3.2 (A)
- net LED_99 renamed LED_B75
- net LED_B75: now also D3.2 (A); no longer D4.2 (A)
- new net: D8.1 (K), R13.1
- new net: D9.1 (K), R14.1
- new net: D7.1 (K), R12.1
- new net: J3.8 (Pin_8), J6.1 (Pin_1), R10.1, R11.1
- new net +5V: J4.29 (Pin_29), J5.8 (Pin_8)
- new net DI_CHARGING: J4.15 (Pin_15), J5.4 (Pin_4)
- new net LED_B99: D4.2 (A), J4.14 (Pin_14)
- new net TP_B+: J5.5 (Pin_5)
- new net TP_B-: J5.6 (Pin_6)
- new net TP_IN+: J2.4 (Pin_4), J5.1 (Pin_1)
- new net TP_IN-: J2.1 (Pin_1), J5.2 (Pin_2)
Other:
- note added: "GND del USB-C"
- note added: "IMPORTANTE: DO_5V es una salida lógica del uC de 3.3v. Hacer un circuito básico que controle el paso o corte de voltaje aquí. Casi siempre estará cortado y sólo se permitirá el voltaje por máximo 10 segundos continuos. Se puede usar un Relé, MOSFET lógico, transistor, o lo que haya."
- note added: "IMPORTANTE: Display catodo común."
- note added: "IMPORTANTE: El USB-C debe sobre salir de la placa un poco (la carsa 3D se hará a la medida de esta placa y se dejará un agujero en ese lugar)"
- note added: "IMPORTANTE: En el diseño final estos elemntos estarán en la capa de ABAJO: - Lector de MicroSD - Push Reset (la idea es que se presione con un palillo por un agujero)"
- note added: "IMPORTANTE: En el diseño final estos elemntos estarán en la capa de arriba: - Display 7 segmentos - Leds (x4) - Push Button (In & Out) - Barra de 5 segmentos led (batería)"
- note added: "IMPORTANTE: En el diseño final estos elemntos estarán en un lado: - Clamp Connections (por un lado) - Conector tipo C (por el otro)"
- note added: "IMPORTANTE: Este botón es parte del esquematico original del STM32. Puedes extender sus terminales a otro lugar y poner un PUSH o puedes dejar este push para reiniciar el micro. Recuerda que se debe presionar con un palo y a veces es metálico así que podrían hacer corto en algún lado."
- note added: "IMPORTANTE: Para TP_B- y TP_B+ dejar headers para soldar los cables de la batería."
- note added: "IMPORTANTE: Si el microSD no aparece como componente se puede armar, sólo ocupa 4 resistencia y 2 capacitores (y el sócalo)."
- note added: "VCC del USB-C"
- note removed: "IMPORTANTE: En el diseño final estos elemntos estarán en la capa de ABAJO: - Lector de MicroSD - Push Reset"
- note removed: "IMPORTANTE: En el diseño final estos elemntos estarán en la capa de arriba: - Display 7 segmentos - Leds - Push Button (In & Out)"
- moved on the sheet: D1, D2, D3, D4, R1, R4, R5, R6, R7, SW3
